Commit message: Tagged vertical surfaces

File: urdf/ceiling.urdf.xacro (robot description, xacro)
@@ -12,17 +12,17 @@
   </joint>
   <xacro:ar_camera parent="ceiling" suffix="0">
-    <origin xyz="-3.81 -5.01 0" rpy="0 0 ${PI}" />
+    <origin xyz="-3.82 -4.97 0" rpy="0 0 ${PI}" />
   </xacro:ar_camera>
   <xacro:ar_camera parent="ceiling" suffix="1">
-    <origin xyz="-2.70 -5.01 0" rpy="0 0 ${PI}" />
+    <origin xyz="-2.60 -4.97 0" rpy="0 0 ${PI}" />
   </xacro:ar_camera>
   <xacro:ar_camera parent="ceiling" suffix="2">
-    <origin xyz="-3.81 -3.79 0" rpy="0 0 ${PI}" />
+    <origin xyz="-3.82 -3.75 0" rpy="0 0 ${PI}" />
   </xacro:ar_camera>
   <xacro:ar_camera parent="ceiling" suffix="3">
-    <origin xyz="-2.70 -3.79 0" rpy="0 0 ${PI}" />
+    <origin xyz="-2.60 -3.75 0" rpy="0 0 ${PI}" />
   </xacro:ar_camera>
   <xacro:ar_camera parent="ceiling" suffix="4">
-    <origin xyz="-3.81 -2.57 0" rpy="0 0 ${PI}" />
+    <origin xyz="-3.82 -2.53 0" rpy="0 0 ${PI}" />
   </xacro:ar_camera>
 </robot>

Commit message: Bundle adjustements

File: urdf/ceiling.urdf.xacro (robot description, xacro)
@@ -9,5 +9,6 @@
     <parent link="map"/>
     <child link="ceiling"/>
-    <origin xyz="6.225 6.625 2.692" rpy="${PI} 0 ${PI_OVER_2}" />
+    <!--<origin xyz="6.225 6.625 2.692" rpy="${PI} 0 ${PI_OVER_2}" />-->
+    <origin xyz="6.1 6.5 2.692" rpy="${PI} 0 ${PI_OVER_2}" />
   </joint>
   <xacro:ar_camera parent="ceiling" suffix="0">

Commit message: Update camera transforms

File: urdf/ceiling.urdf.xacro (robot description, xacro)
@@ -13,17 +13,17 @@
   </joint>
   <xacro:ar_camera parent="ceiling" suffix="0">
-    <origin xyz="-3.82 -4.97 0" rpy="0 0 ${PI}" />
+    <origin xyz="-3.19 -5.065 0" rpy="0 0 0" />
   </xacro:ar_camera>
   <xacro:ar_camera parent="ceiling" suffix="1">
-    <origin xyz="-2.60 -4.97 0" rpy="0 0 ${PI}" />
+    <origin xyz="-3.48 -3.925 0" rpy="0 0 ${PI_OVER_2}" />
   </xacro:ar_camera>
   <xacro:ar_camera parent="ceiling" suffix="2">
-    <origin xyz="-3.82 -3.75 0" rpy="0 0 ${PI}" />
+    <origin xyz="-4.14 -3.01 0" rpy="0 0 -${PI_OVER_2}" />
   </xacro:ar_camera>
   <xacro:ar_camera parent="ceiling" suffix="3">
-    <origin xyz="-2.60 -3.75 0" rpy="0 0 ${PI}" />
+    <origin xyz="-2.90 -2.25 0" rpy="0 0 -${PI_OVER_2}" />
   </xacro:ar_camera>
   <xacro:ar_camera parent="ceiling" suffix="4">
-    <origin xyz="-3.82 -2.53 0" rpy="0 0 ${PI}" />
+    <origin xyz="-3.70 -0.84 0" rpy="0 0 0" />
   </xacro:ar_camera>
 </robot>

Commit message: Camera transform adjustements

File: urdf/ceiling.urdf.xacro (robot description, xacro)
@@ -13,11 +13,11 @@
   </joint>
   <xacro:ar_camera parent="ceiling" suffix="0">
-    <origin xyz="-3.19 -5.065 0" rpy="0 0 0" />
+    <origin xyz="-2.96 -5.05 0" rpy="0 0 0" />
   </xacro:ar_camera>
   <xacro:ar_camera parent="ceiling" suffix="1">
-    <origin xyz="-3.48 -3.925 0" rpy="0 0 ${PI_OVER_2}" />
+    <origin xyz="-3.37 -3.83 0" rpy="0 0 ${PI_OVER_2}" />
   </xacro:ar_camera>
   <xacro:ar_camera parent="ceiling" suffix="2">
-    <origin xyz="-4.14 -3.01 0" rpy="0 0 -${PI_OVER_2}" />
+    <origin xyz="-3.82 -3.01 0" rpy="0 0 -${PI_OVER_2}" />
   </xacro:ar_camera>
   <xacro:ar_camera parent="ceiling" suffix="3">

Commit message: Fixed transform from map to ceiling

File: urdf/ceiling.urdf.xacro (robot description, xacro)
@@ -9,6 +9,6 @@
     <parent link="map"/>
     <child link="ceiling"/>
-    <!--<origin xyz="6.225 6.625 2.692" rpy="${PI} 0 ${PI_OVER_2}" />-->
-    <origin xyz="6.1 6.5 2.692" rpy="${PI} 0 ${PI_OVER_2}" />
+    <!--<origin xyz="6.1 6.5 2.692" rpy="${PI} 0 ${PI_OVER_2}" />-->
+    <origin xyz="0.55 6.34 2.692" rpy="${PI} 0 -${PI}" />
   </joint>
   <xacro:ar_camera parent="ceiling" suffix="0">

Commit message: Fixed transforms

File: urdf/ceiling.urdf.xacro (robot description, xacro)
@@ -22,8 +22,8 @@
   </xacro:ar_camera>
   <xacro:ar_camera parent="ceiling" suffix="3">
-    <origin xyz="-2.90 -2.25 0" rpy="0 0 -${PI_OVER_2}" />
+    <origin xyz="-2.80 -2.30 0" rpy="0 0 -${PI_OVER_2}" />
   </xacro:ar_camera>
   <xacro:ar_camera parent="ceiling" suffix="4">
-    <origin xyz="-3.70 -0.84 0" rpy="0 0 0" />
+    <origin xyz="-3.80 -0.90 0" rpy="0 0 0" />
   </xacro:ar_camera>
 </robot>

Commit message: Added option to stop publishing maps while driving

File: urdf/ceiling.urdf.xacro (robot description, xacro)
@@ -9,18 +9,18 @@
     <parent link="map"/>
     <child link="ceiling"/>
-    <!--<origin xyz="6.1 6.5 2.692" rpy="${PI} 0 ${PI_OVER_2}" />-->
-    <origin xyz="0.55 6.34 2.692" rpy="${PI} 0 -${PI}" />
+    <!--<origin xyz="0.55 6.34 2.692" rpy="${PI} 0 -${PI}" />-->
+    <origin xyz="0.35 6.36 2.692" rpy="${PI} 0 -${PI}" />
   </joint>
   <xacro:ar_camera parent="ceiling" suffix="0">
-    <origin xyz="-2.96 -5.05 0" rpy="0 0 0" />
+    <origin xyz="-3.10 -5.17 0" rpy="0 0 0" />
   </xacro:ar_camera>
   <xacro:ar_camera parent="ceiling" suffix="1">
-    <origin xyz="-3.37 -3.83 0" rpy="0 0 ${PI_OVER_2}" />
+    <origin xyz="-3.55 -3.83 0" rpy="0 0 ${PI_OVER_2}" />
   </xacro:ar_camera>
   <xacro:ar_camera parent="ceiling" suffix="2">
-    <origin xyz="-3.82 -3.01 0" rpy="0 0 -${PI_OVER_2}" />
+    <origin xyz="-3.98 -3.08 0" rpy="0 0 -${PI_OVER_2}" />
   </xacro:ar_camera>
   <xacro:ar_camera parent="ceiling" suffix="3">
-    <origin xyz="-2.80 -2.30 0" rpy="0 0 -${PI_OVER_2}" />
+    <origin xyz="-2.95 -2.28 0" rpy="0 0 -${PI_OVER_2}" />
   </xacro:ar_camera>
   <xacro:ar_camera parent="ceiling" suffix="4">
